File: designs/hardware/ESP32 nGeigieNano WiFi/bGeigieCast_V1.4.0.kicad_pcb (KiCad board)
At the start: 2 copper layers, 25.5 x 32 mm, 10 parts, among them SW1 TACT-SWITCH, SW2 SWITCH_INV, U1 ESP32S, U2 XBEE-socket

Commit message: Added bGigeiCast files to be implemented
Other:
- net class Default removed
- net class Power removed
