File: designs/hardware/ESP32 nGeigieNano WiFi/xbee.kicad_pcb (KiCad board)
At the start: 2 copper layers, 25.5 x 32 mm, 10 parts, among them SW1 TACT-SWITCH, SW2 SWITCH_INV, U1 ESP32S, U2 XBEE-socket

Commit message: New branch for M5stamp pico
Other:
- board text added: "bGeigie-Cast V1.4.0 SAFECAST 2021"
- board text removed: "bGeigie-Cast V1.4.0 SAFECAST 2019"
