File: designs/hardware/ESP32 nGeigieNano WiFi/xbee.kicad_pcb (KiCad board)
At the start: 2 copper layers, 25.5 x 32 mm, 10 parts, among them SW1 TACT-SWITCH, SW2 SWITCH_INV, U1 ESP32S, U2 XBEE-socket

Commit message: d V1.6.0 boards
Parts:
- C1: value CP1 -> 330uF
Connections:
- SW2 pad 3: (no net) -> unconnected-(SW2-C-Pad3)
- U1 pad 11: (no net) -> unconnected-(U1-IO26-Pad11)
- U1 pad 12: (no net) -> unconnected-(U1-IO27-Pad12)
- U1 pad 13: (no net) -> unconnected-(U1-IO14-Pad13)
- U1 pad 14: (no net) -> unconnected-(U1-IO12-Pad14)
- U1 pad 16: (no net) -> unconnected-(U1-IO13-Pad16)
- U1 pad 17: (no net) -> unconnected-(U1-SD2/IO9-Pad17)
- U1 pad 18: (no net) -> unconnected-(U1-SD3/IO10-Pad18)
- U1 pad 19: (no net) -> unconnected-(U1-CMD/IO11-Pad19)
- U1 pad 20: (no net) -> unconnected-(U1-CLK/IO6-Pad20)
- U1 pad 21: (no net) -> unconnected-(U1-SD0/IO7-Pad21)
- U1 pad 22: (no net) -> unconnected-(U1-SD1/IO8-Pad22)
- U1 pad 23: (no net) -> unconnected-(U1-IO15-Pad23)
- U1 pad 24: (no net) -> unconnected-(U1-IO2-Pad24)
- U1 pad 26: (no net) -> unconnected-(U1-IO4-Pad26)
- U1 pad 28: (no net) -> unconnected-(U1-IO17-Pad28)
- U1 pad 29: (no net) -> unconnected-(U1-IO5-Pad29)
- U1 pad 30: (no net) -> unconnected-(U1-IO18-Pad30)
- U1 pad 31: (no net) -> unconnected-(U1-IO19-Pad31)
- U1 pad 32: (no net) -> unconnected-(U1-NC-Pad32)
- U1 pad 33: (no net) -> unconnected-(U1-IO21-Pad33)
- U1 pad 36: (no net) -> unconnected-(U1-IO22-Pad36)
- U1 pad 37: (no net) -> unconnected-(U1-IO23-Pad37)
- U1 pad 38: (no net) -> unconnected-(U1-GND-Pad38)
- U1 pad 4: (no net) -> unconnected-(U1-SENSOR_VP-Pad4)
- U1 pad 5: (no net) -> unconnected-(U1-SENSOR_VN-Pad5)
- U1 pad 6: (no net) -> unconnected-(U1-IO34-Pad6)
- U1 pad 7: (no net) -> unconnected-(U1-IO35-Pad7)
- U2 pad 11: (no net) -> unconnected-(U2-DIO4-Pad11)
- U2 pad 12: (no net) -> unconnected-(U2-CTS-Pad12)
- U2 pad 13: (no net) -> unconnected-(U2-DIO9-Pad13)
- U2 pad 14: (no net) -> unconnected-(U2-RES@14-Pad14)
- U2 pad 15: (no net) -> unconnected-(U2-DIO5-Pad15)
- U2 pad 16: (no net) -> unconnected-(U2-RTS-Pad16)
- U2 pad 17: (no net) -> unconnected-(U2-DIO3-Pad17)
- U2 pad 18: (no net) -> unconnected-(U2-DIO2-Pad18)
- U2 pad 19: (no net) -> unconnected-(U2-DIO1-Pad19)
- U2 pad 20: (no net) -> unconnected-(U2-DIO0-Pad20)
- U2 pad 4: (no net) -> unconnected-(U2-DIO12-Pad4)
- U2 pad 5: (no net) -> unconnected-(U2-RESET-Pad5)
- U2 pad 6: (no net) -> unconnected-(U2-RSSI-Pad6)
- U2 pad 7: (no net) -> unconnected-(U2-DIO11-Pad7)
- U2 pad 8: (no net) -> unconnected-(U2-RES@8-Pad8)
- U2 pad 9: (no net) -> unconnected-(U2-DTR-Pad9)
