File: designs/hardware/bGeigieCast V1.5.0 (ESP32-C3)/bGeigieCast V1.5.kicad_pcb (KiCad board)
At the start: 2 copper layers, 25.5 x 32 mm, 10 parts, among them SW1 TACT-SWITCH, SW2 SWITCH_INV, U1 ESP32S, U2 XBEE-socket

Commit message: V1.5.0 with ESP32-C3
Parts:
- removed U1: ESP32S, ESP32-footprints-Lib:ESP-32S
- added IC1: ESP32-C3-WROOM-02-N4, ESP32-C3-WROOM-02-N4:ESP32C3WROOM02N4, F.Cu at (149.4, 106.4)
- C1: value CP1 -> 330uF
Connections:
- SW2 pad 3: (no net) -> unconnected-(SW2-Pad3)
- U2 pad 11: (no net) -> unconnected-(U2-Pad11)
- U2 pad 12: (no net) -> unconnected-(U2-Pad12)
- U2 pad 13: (no net) -> unconnected-(U2-Pad13)
- U2 pad 14: (no net) -> unconnected-(U2-Pad14)
- U2 pad 15: (no net) -> unconnected-(U2-Pad15)
- U2 pad 16: (no net) -> unconnected-(U2-Pad16)
- U2 pad 17: (no net) -> unconnected-(U2-Pad17)
- U2 pad 18: (no net) -> unconnected-(U2-Pad18)
- U2 pad 19: (no net) -> unconnected-(U2-Pad19)
- U2 pad 20: (no net) -> unconnected-(U2-Pad20)
- U2 pad 4: (no net) -> unconnected-(U2-Pad4)
- U2 pad 5: (no net) -> unconnected-(U2-Pad5)
- U2 pad 6: (no net) -> unconnected-(U2-Pad6)
- U2 pad 7: (no net) -> unconnected-(U2-Pad7)
- U2 pad 8: (no net) -> unconnected-(U2-Pad8)
- U2 pad 9: (no net) -> unconnected-(U2-Pad9)
Routing:
- net GND: track 54.2 -> 0.00 mm, vias 4 -> 0
- net Net-(U2-Pad3): track 51.6 -> 0.00 mm
- net VDD: track 39.9 -> 0.00 mm
- net +3V3: track 30.8 -> 0.00 mm, vias 2 -> 0
- net Net-(U2-Pad2): track 21.1 -> 0.00 mm, vias 1 -> 0
- net Net-(D1-Pad4): track 19.9 -> 0.00 mm, vias 1 -> 0
- net Net-(SW1-Pad1): track 16.9 -> 0.00 mm
- net Net-(D1-Pad1): track 8.96 -> 0.00 mm, vias 1 -> 0
- net Net-(R4-Pad1): track 8.57 -> 0.00 mm, vias 1 -> 0
- net Net-(D1-Pad3): track 8.22 -> 0.00 mm, vias 1 -> 0
- net Net-(R3-Pad1): track 7.65 -> 0.00 mm, vias 1 -> 0
- net Net-(R1-Pad1): track 5.57 -> 0.00 mm, vias 1 -> 0
