File: designs/hardware/bGeigieCastV1.5.0 (ESP32-C3)/bGeigieCastV1.5.kicad_pcb (KiCad board)
At the start: 2 copper layers, 25.5 x 32 mm, 10 parts, among them SW1 TACT-SWITCH, SW2 SWITCH_INV, U1 ESP32S, U2 XBEE-socket

Commit message: Updated board V1.5.0
Parts:
- removed G***: LOGO, ESP32 nGeigieNano WiFi all:QR_code_safecast_bgc
- added U3: ESP32-C3, RF_Module:ESP-12E, F.Cu at (176.7, 107.0)
- C1: value CP1 -> 330uF
Connections:
- SW2 pad 3: (no net) -> unconnected-(SW2-Pad3)
- U1 pad 11: (no net) -> unconnected-(U1-Pad11)
- U1 pad 12: (no net) -> unconnected-(U1-Pad12)
- U1 pad 13: (no net) -> unconnected-(U1-Pad13)
- U1 pad 14: (no net) -> unconnected-(U1-Pad14)
- U1 pad 16: (no net) -> unconnected-(U1-Pad16)
- U1 pad 17: (no net) -> unconnected-(U1-Pad17)
- U1 pad 18: (no net) -> unconnected-(U1-Pad18)
- U1 pad 19: (no net) -> unconnected-(U1-Pad19)
- U1 pad 20: (no net) -> unconnected-(U1-Pad20)
- U1 pad 21: (no net) -> unconnected-(U1-Pad21)
- U1 pad 22: (no net) -> unconnected-(U1-Pad22)
- U1 pad 23: (no net) -> unconnected-(U1-Pad23)
- U1 pad 24: (no net) -> unconnected-(U1-Pad24)
- U1 pad 26: (no net) -> unconnected-(U1-Pad26)
- U1 pad 28: (no net) -> unconnected-(U1-Pad28)
- U1 pad 29: (no net) -> unconnected-(U1-Pad29)
- U1 pad 30: (no net) -> unconnected-(U1-Pad30)
- U1 pad 31: (no net) -> unconnected-(U1-Pad31)
- U1 pad 32: (no net) -> unconnected-(U1-Pad32)
- U1 pad 33: (no net) -> unconnected-(U1-Pad33)
- U1 pad 36: (no net) -> unconnected-(U1-Pad36)
- U1 pad 37: (no net) -> unconnected-(U1-Pad37)
- U1 pad 38: (no net) -> unconnected-(U1-Pad38)
- U1 pad 4: (no net) -> unconnected-(U1-Pad4)
- U1 pad 5: (no net) -> unconnected-(U1-Pad5)
- U1 pad 6: (no net) -> unconnected-(U1-Pad6)
- U1 pad 7: (no net) -> unconnected-(U1-Pad7)
- U2 pad 11: (no net) -> unconnected-(U2-Pad11)
- U2 pad 12: (no net) -> unconnected-(U2-Pad12)
- U2 pad 13: (no net) -> unconnected-(U2-Pad13)
- U2 pad 14: (no net) -> unconnected-(U2-Pad14)
- U2 pad 15: (no net) -> unconnected-(U2-Pad15)
- U2 pad 16: (no net) -> unconnected-(U2-Pad16)
- U2 pad 17: (no net) -> unconnected-(U2-Pad17)
- U2 pad 18: (no net) -> unconnected-(U2-Pad18)
- U2 pad 19: (no net) -> unconnected-(U2-Pad19)
- U2 pad 20: (no net) -> unconnected-(U2-Pad20)
- U2 pad 4: (no net) -> unconnected-(U2-Pad4)
- U2 pad 5: (no net) -> unconnected-(U2-Pad5)
- U2 pad 6: (no net) -> unconnected-(U2-Pad6)
- U2 pad 7: (no net) -> unconnected-(U2-Pad7)
- U2 pad 8: (no net) -> unconnected-(U2-Pad8)
- U2 pad 9: (no net) -> unconnected-(U2-Pad9)
Other:
- board text added: "Scan QR code for manual bGeigie-Cast V1.5.0 info@safecast.org"
- board text added: "bGeigie-Cast V1.5.0 SAFECAST 2021"
- board text removed: "Scan QR code for manual bGeigie-Cast V1.4.0 info@safecast.org"
- board text removed: "bGeigie-Cast V1.4.0 SAFECAST 2019"

Commit message: Update
Parts:
- removed U1: ESP32S, ESP32-footprints-Lib:ESP-32S
- U3: value ESP32-C3 -> ESP-12E
- moved U3 29.1 mm to (148.1, 101.3)
Connections:
- SW1 pad 1: Net-(SW1-Pad1) -> Net-(U3-Pad18)
- U2 pad 2: Net-(U1-Pad35) -> Net-(U3-Pad21)
- U2 pad 3: Net-(U1-Pad27) -> Net-(U3-Pad22)
- U3 pad 15: unconnected-(U3-Pad15) -> GND
- U3 pad 17: (no net) -> unconnected-(U3-Pad17)
- U3 pad 18: (no net) -> Net-(U3-Pad18)
- U3 pad 19: (no net) -> unconnected-(U3-Pad19)
- U3 pad 20: (no net) -> unconnected-(U3-Pad20)
- U3 pad 21: (no net) -> Net-(U3-Pad21)
- U3 pad 22: (no net) -> Net-(U3-Pad22)
- U3 pad 3: unconnected-(U3-Pad3) -> +3V3
- U3 pad 5: unconnected-(U3-Pad5) -> Net-(R1-Pad1)
- U3 pad 6: unconnected-(U3-Pad6) -> Net-(R4-Pad1)
- U3 pad 7: unconnected-(U3-Pad7) -> Net-(R3-Pad1)
- U3 pad 8: unconnected-(U3-Pad8) -> +3V3
Routing:
- net GND: track 54.2 -> 2.14 mm, vias 4 -> 1
- net Net-(U1-Pad27): track 51.6 -> 0.00 mm
- net Net-(U3-Pad22): track 0.00 -> 25.4 mm
- net Net-(U3-Pad18): track 0.00 -> 23.2 mm
- net Net-(U1-Pad35): track 21.1 -> 0.00 mm, vias 1 -> 0
- net Net-(U3-Pad21): track 0.00 -> 19.0 mm
- net Net-(SW1-Pad1): track 16.9 -> 0.00 mm
- net VDD: track 39.9 -> 24.9 mm
- net Net-(D1-Pad4): track 19.9 -> 13.0 mm
- net +3V3: track 30.8 -> 24.6 mm, vias 2 -> 1
- net Net-(R3-Pad1): track 7.65 -> 4.32 mm
- net Net-(D1-Pad3): track 8.22 -> 7.51 mm
- net Net-(D1-Pad1): track 8.96 -> 9.64 mm
Other:
- board text added: "Scan QR code for manual bGeigieCast V1.5.0 info@safecast.org"
- board text added: "bGeigieCast V1.5.0 SAFECAST 2021"
- board text removed: "Scan QR code for manual bGeigie-Cast V1.5.0 info@safecast.org"
- board text removed: "bGeigie-Cast V1.5.0 SAFECAST 2021"
