File: designs/hardware/bGeigieCastV1.5.0 (ESP32-C3)/bGeigieCastV1.5.kicad_sch (KiCad schematic)
At the start: 9 parts, among them SW1 TACT-SWITCH, SW2 SWITCH_INV, U1 ESP32S, U2 XBEE-socket

Commit message: Updated board V1.5.0
Parts:
- added U3: WeMos_D1_mini, RF_Module:ESP-12E, symbol MCU_Module:WeMos_D1_mini
Other:
- note added: "V1.5.0"
- note added: "bGeigieNano ESP32 Xbee V1.5.0"
- note removed: "V1.1"
- note removed: "bGeigieNano ESP32 Xbee V1.4.0"
Changed lines of the file:
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@@
 (kicad_sch (version 20210621) (generator eeschema)
   (paper "A4")
+  (title_block
+    (date "2021-07-22")
+    (rev "V1.5.0")
+  )
   (junction (at 80.01 60.96) (diameter 0.259) (color 0 0 0 0))
   (junction (at 87.63 50.8) (diameter 0.259) (color 0 0 0 0))
@@
     (stroke (width 0) (type solid) (color 0 0 0 0))
   )
-  (text "bGeigieNano ESP32 Xbee V1.4.0" (at 186.69 190.5 0)
+  (text "bGeigieNano ESP32 Xbee V1.5.0" (at 186.69 190.5 0)
     (effects (font (size 1.27 1.27)) (justify left bottom))
   )
@@
     (effects (font (size 1.27 1.27)) (justify left bottom))
   )
-  (text "V1.1" (at 269.24 194.31 0)
+  (text "V1.5.0" (at 269.24 194.31 0)
     (effects (font (size 1.27 1.27)) (justify left bottom))
   )
@@
     (pin "3")
     (pin "4")
+  )
+  (symbol (lib_id "MCU_Module:WeMos_D1_mini") (at 50.8 93.98 0) (unit 1)
+    (in_bom yes) (on_board yes) (fields_autoplaced)
+    (property "Reference" "U3" (id 0) (at 50.8 116.7036 0))
+    (property "Value" "WeMos_D1_mini" (id 1) (at 50.8 119.4787 0))
+    (property "Footprint" "RF_Module:ESP-12E" (id 2) (at 50.8 123.19 0)
+      (effects (font (size 1.27 1.27)) hide)
+    )
+    (property "Datasheet" "https://wiki.wemos.cc/products:d1:d1_mini#documentation" (id 3) (at 3.81 123.19 0)
+      (effects (font (size 1.27 1.27)) hide)
+    )
+    (pin "1")
+    (pin "10")
+    (pin "11")
+    (pin "12")
+    (pin "13")
+    (pin "14")
+    (pin "15")
+    (pin "16")
+    (pin "2")
+    (pin "3")
+    (pin "4")
+    (pin "5")
+    (pin "6")
+    (pin "7")
+    (pin "8")
+    (pin "9")
   )
   (symbol (lib_id "xbee-eagle-import:XBEE-1B2") (at 113.03 129.54 180) (unit 1)
@@
       (reference "U2") (unit 1) (value "XBEE-socket") (footprint "digikey-footprints:XBEE-20_THT")
     )
-  )
+    (path "/78d23029-2d20-4e11-88de-437c6f9563b5"
+      (reference "U3") (unit 1) (value "WeMos_D1_mini") (footprint "RF_Module:ESP-12E")
+    )
+  )

Commit message: Update
Parts:
- removed U1: ESP32S, ESP32-footprints-Lib:ESP-32S, symbol xbee-rescue:ESP32S-espressif-xess
- removed U3: WeMos_D1_mini, RF_Module:ESP-12E, symbol MCU_Module:WeMos_D1_mini
- added U3: ESP-12E, RF_Module:ESP-12E, symbol RF_Module:ESP-12E
Connections:
- net +3V3: now also U3.3 (EN), U3.8 (VCC)
- net GND: now also U3.15 (GND)
- net at U2.2 (DOUT): now also U3.21 (GPIO3/RXD)
- net at U2.3 (DIN): now also U3.22 (GPIO1/TXD)
- net at SW1.1: now also U3.18 (GPIO0)
- net at R1.1: now also U3.4 (GPIO16)
- net at R3.1: now also U3.5 (GPIO14)
- net at R4.1: now also U3.7 (GPIO13)
Other:
- moved on the sheet: C1, U2
