File: designs/hardware/bGeigieCast V1.6.0(StampS3)/bGeigieCast V1.6.0(StampS3)/bGeigieCast V1.6.0(StampS3).kicad_sch (KiCad schematic)
At the start: 4 parts, among them J1 Left, J2 Right, U1 ESP-12, U2 XBEE-socket

Commit message: Added V1.6.2 Gerbers and many boards updates.
Parts:
- removed U1: ESP-12, ESP8266:ESP-12, symbol ESP8266:ESP-12
- J1: footprint Connector_PinHeader_2.54mm:PinHeader_1x06_P2.54mm_Vertical -> Connector_PinHeader_2.54mm:PinHeader_1x09_P2.54mm_Vertical
Connections:
- net +3.3V: now reaches J2.7 (Pin_7), U2.1 (VDD)
- net at J1.3 (Pin_4): no longer U2.10 (GND)
- net at U2.2 (DOUT): now also J2.8 (Pin_8); no longer J1.1 (Pin_6)
- net at U2.3 (DIN): now also J2.9 (Pin_9); no longer J1.2 (Pin_5)
- net GND: now reaches J2.12 (Pin_12)
- net GND: now also U2.10 (GND)
Other:
- note added: "bGeigieCast M5stack Stamp V1.6.1"
- note removed: "2019-06-24"
- note removed: "bGeigieNano ESP32 Xbee V1.4.0"
- moved on the sheet: J1, J2, U2
